Commit message: update diffRobot URDF

File: src/diffRobot/urdf/diffRobot.urdf.xacro (robot description, xacro)
@@ -1,17 +1,25 @@
-<robot xmlns:xacro="http://www.ros.org/wiki/xacro" name="diffRobot">
-    <link name="base_footprint"></link>
+<?xml version='1.0'?>
+<robot name="diffrobot" xmlns:xacro="http://www.ros.org/wiki/xacro">
+    <!-- <xacro:include filename="$(find diffrobot_description)/urdf/diffrobot.gazebo"/> -->
+    <link name="base_footprint"/>
+    <joint name="robot_footprint_joint" type="fixed">
+        <origin xyz="0 0 0.0" rpy="0 0 0" />
+        <parent link="base_footprint"/>
+        <child link="base_link"/>
+    </joint>
     <link name="base_link">
         <inertial>
             <origin xyz="0.0 0.0 0.0" rpy="0.0 0.0 0.0"/>
-            <mass value="0.0"/>
+            <mass value="5.0"/>
+            <inertia ixx="0.0" ixy="0.0" ixz="0.0" iyy="0.0" iyz="0.0" izz="0.0"/>
         </inertial>
-        <visual name="base_link">
+        <visual name="base_link_visual">
             <origin xyz="0.0 0.0 0.0" rpy="0.0 0.0 0.0"/>
             <geometry>
-                <box size="0.0 0.0 0.0"/>
+                <box size="0.4 0.2 0.1"/>
             </geometry>
             <material name="">
-                <color rgba="1.0 0.0 0.0 1.0"/>
-                <texture filename="base_link"/>
+                <color rgba="0.0 0.0 1.0 1.0"/>
+                <texture filename=""/>
             </material>
         </visual>
@@ -19,52 +27,115 @@
             <origin xyz="0.0 0.0 0.0" rpy="0.0 0.0 0.0"/>
             <geometry>
-                <box size="0.0 0.0 0.0"/>
+                <box size="0.4 0.2 0.1"/>
             </geometry>
         </collision>
     </link>
-    <link name="wheel_left">
-        <visual>
+    <link name="left_wheel">
+        <inertial>
+            <origin xyz="0.0 0.0 0.0" rpy="0.0 1.5707 1.5707"/>
+            <mass value="5.0"/>
+            <inertia ixx="0.1" ixy="0.0" ixz="0.0" iyy="0.1" iyz="0.0" izz="0.1"/>
+        </inertial>
+        <visual name="left_wheel_visual">
             <origin xyz="0.0 0.0 0.0" rpy="0.0 0.0 0.0"/>
             <geometry>
-                <sphere radius="0.05" />
+                <cylinder radius="0.1" length="0.05"/>
             </geometry>
         </visual>
-    </link>
-    <link name="wheel_right">
-        <visual>
+        <collision name='left_wheel_collision'>
             <origin xyz="0.0 0.0 0.0" rpy="0.0 0.0 0.0"/>
             <geometry>
-                <sphere radius="0.05" />
+                <cylinder radius="0.1" length="0.05"/>
+            </geometry>
+        </collision>
+    </link>
+    <link name="right_wheel">
+        <inertial>
+            <origin xyz="0.0 0.0 0.0" rpy="0.0 0.0 0.0"/>
+            <mass value="5.0"/>
+            <inertia ixx="0.1" ixy="0.0" ixz="0.0" iyy="0.1" iyz="0.0" izz="0.1"/>
+        </inertial>
+        <visual name="right_wheel_visual">
+            <origin xyz="0.0 0.0 0.0" rpy="0.0 0.0 0.0"/>
+            <geometry>
+                <cylinder radius="0.1" length="0.05"/>
             </geometry>
         </visual>
-    </link>
-    <link name="Caster_wheel">
-        <visual>
+        <collision name='right_wheel_collision'>
             <origin xyz="0.0 0.0 0.0" rpy="0.0 0.0 0.0"/>
             <geometry>
-                <sphere radius="0.05" />
+                <cylinder radius="0.1" length="0.05"/>
             </geometry>
+        </collision>
+    </link>
+    <joint name="wheel_left_joint" type="continuous">
+        <origin xyz="0.0 0.15 0.0" rpy="0.0 1.5705 1.5705"/>
+        <parent link="base_link"/>
+        <child link="left_wheel"/>
+        <axis xyz="0.0 0.0 1.0"/>
+    </joint>
+    <joint name="wheel_right_joint" type="continuous">
+        <origin xyz="0.0 -0.15 0.0" rpy="0.0 1.5705 1.5705"/>
+        <parent link="base_link"/>
+        <child link="right_wheel"/>
+        <axis xyz="0.0 0.0 1.0"/>
+    </joint>
+    <link name="front_caster">
+        <inertial>
+            <origin xyz="0.0 0.0 0.0" rpy="0.0 0.0 0.0"/>
+            <mass value="0.0"/>
+            <inertia ixx="0.0" ixy="0.0" ixz="0.0" iyy="0.0" iyz="0.0" izz="0.0"/>
+        </inertial>
+        <visual name="front_caster_visual">
+            <origin xyz="0.0 0.0 0.0" rpy="0.0 0.0 0.0"/>
+            <geometry>
+                <sphere radius="0.0499"/>
+            </geometry>
+            <material name="">
+                <color rgba="1.0 1.0 1.0 1.0"/>
+                <texture filename=""/>
+            </material>
         </visual>
+        <collision>
+            <origin xyz="0.0 0.0 0.0" rpy="0.0 0.0 0.0"/>
+            <geometry>
+                <sphere radius="0.0499"/>
+            </geometry>
+        </collision>
     </link>
-    <!-- Joints -->
-    <joint name="base_joint" type="fixed"></joint>
-        <origin xyz="0.0 0.0 0.0" rpy="0.0 0.0 0.0"/>
-        <parent link="base_footprint"/>
-        <child link="base_link"/>
+    <joint name="front_caster_joint" type="fixed">
+        <origin xyz="0.15 0.0 -0.05" rpy="0.0 0.0 0.0"/>
+        <parent link="base_link"/>
+        <child link="front_caster"/>
+        <axis xyz="0.0 0.0 0.0"/>
+    </joint>
+ <link name="back_caster">
+        <inertial>
+            <origin xyz="0.0 0.0 0.0" rpy="0.0 0.0 0.0"/>
+            <mass value="0.0"/>
+            <inertia ixx="0.0" ixy="0.0" ixz="0.0" iyy="0.0" iyz="0.0" izz="0.0"/>
+        </inertial>
+        <visual name="back_caster_visual">
+            <origin xyz="0.0 0.0 0.0" rpy="0.0 0.0 0.0"/>
+            <geometry>
+                <sphere radius="0.0499"/>
+            </geometry>
+            <material name="">
+                <color rgba="1.0 1.0 1.0 1.0"/>
+                <texture filename=""/>
+            </material>
+        </visual>
+        <collision>
+            <origin xyz="0.0 0.0 0.0" rpy="0.0 0.0 0.0"/>
+            <geometry>
+                <sphere radius="0.0499"/>
+            </geometry>
+        </collision>
     </link>
-    <joint name="wheel_left_joint" type="revolute">
-        <origin xyz="0.0 0.0 0.0" rpy="0.0 0.0 0.0"/>
+    <joint name="back_caster_joint" type="fixed">
+        <origin xyz="-0.15 0.0 -0.05" rpy="0.0 0.0 0.0"/>
         <parent link="base_link"/>
-        <child link="wheel_left"/>
-    </joint>
-    <joint name="wheel_right_joint" type="revolute">
-        <origin xyz="0.0 0.0 0.0" rpy="0.0 0.0 0.0"/>
-        <parent link="base_link"/>
-        <child link="wheel_right"/>
-    </joint>
-    <joint name="caster_wheel_joint" type="fixed">
-        <origin xyz="0.0 0.0 0.0" rpy="0.0 0.0 0.0"/>
-        <parent link="base_link"/>
-        <child link="caster_wheel"/>
+        <child link="back_caster"/>
+        <axis xyz="0.0 0.0 0.0"/>
     </joint>
 </robot>
